File: ElectroChessboard1/BoardHalls2.kicad_sch (KiCad schematic)
At the start: 18 parts, among them IC19 A3213ELHLT-T, IC20 A3213ELHLT-T, IC21 A3213ELHLT-T, IC22 A3213ELHLT-T, IC23 A3213ELHLT-T, IC24 A3213ELHLT-T, IC25 A3213ELHLT-T, IC26 A3213ELHLT-T, IC27 A3213ELHLT-T, IC28 A3213ELHLT-T, IC29 A3213ELHLT-T, IC30 A3213ELHLT-T, IC31 A3213ELHLT-T, IC32 A3213ELHLT-T, IC33 A3213ELHLT-T, IC34 A3213ELHLT-T, IC35 ADG708BRUZ-REEL7, IC36 ADG708BRUZ-REEL7

Commit message: Corrected footprints 1
Chosen footprints for JLCPCB
I may add USB insterface chip
Parts:
- IC19, IC20, IC21, IC22, IC23, IC24, IC25, IC26, IC27, IC28, IC29, IC30, IC31, IC32, IC33, IC34: footprint A3213ELHLTT -> SamacSys_Parts:A3213ELHLTT
- IC35, IC36: footprint SOP65P640X120-16N -> SamacSys_Parts:SOP65P640X120-16N
Changed lines of the file:
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@@
 			)
 		)
-		(property "Footprint" "A3213ELHLTT"
+		(property "Footprint" "SamacSys_Parts:A3213ELHLTT"
 			(at 87.96 152.4 0)
 			(effects
@@
 			)
 		)
-		(property "Footprint" "A3213ELHLTT"
+		(property "Footprint" "SamacSys_Parts:A3213ELHLTT"
 			(at 15.57 80.01 0)
 			(effects
@@
 			)
 		)
-		(property "Footprint" "A3213ELHLTT"
+		(property "Footprint" "SamacSys_Parts:A3213ELHLTT"
 			(at 66.37 80.01 0)
 			(effects
@@
 			)
 		)
-		(property "Footprint" "A3213ELHLTT"
+		(property "Footprint" "SamacSys_Parts:A3213ELHLTT"
 			(at -35.23 80.01 0)
 			(effects
@@
 			)
 		)
-		(property "Footprint" "A3213ELHLTT"
+		(property "Footprint" "SamacSys_Parts:A3213ELHLTT"
 			(at 37.16 152.4 0)
 			(effects
@@
 			)
 		)
-		(property "Footprint" "SOP65P640X120-16N"
+		(property "Footprint" "SamacSys_Parts:SOP65P640X120-16N"
 			(at 243.84 196.52 0)
 			(effects
@@
 			)
 		)
-		(property "Footprint" "A3213ELHLTT"
+		(property "Footprint" "SamacSys_Parts:A3213ELHLTT"
 			(at 40.97 80.01 0)
 			(effects
@@
 			)
 		)
-		(property "Footprint" "A3213ELHLTT"
+		(property "Footprint" "SamacSys_Parts:A3213ELHLTT"
 			(at 62.56 152.4 0)
 			(effects
@@
 			)
 		)
-		(property "Footprint" "A3213ELHLTT"
+		(property "Footprint" "SamacSys_Parts:A3213ELHLTT"
 			(at 91.77 80.01 0)
 			(effects
@@
 			)
 		)
-		(property "Footprint" "A3213ELHLTT"
+		(property "Footprint" "SamacSys_Parts:A3213ELHLTT"
 			(at -9.83 80.01 0)
 			(effects
@@
 			)
 		)
-		(property "Footprint" "A3213ELHLTT"
+		(property "Footprint" "SamacSys_Parts:A3213ELHLTT"
 			(at -39.04 152.4 0)
 			(effects
@@
 			)
 		)
-		(property "Footprint" "A3213ELHLTT"
+		(property "Footprint" "SamacSys_Parts:A3213ELHLTT"
 			(at 113.36 152.4 0)
 			(effects
@@
 			)
 		)
-		(property "Footprint" "A3213ELHLTT"
+		(property "Footprint" "SamacSys_Parts:A3213ELHLTT"
 			(at -13.64 152.4 0)
 			(effects
@@
 			)
 		)
-		(property "Footprint" "A3213ELHLTT"
+		(property "Footprint" "SamacSys_Parts:A3213ELHLTT"
 			(at -64.44 152.4 0)
 			(effects
@@
 			)
 		)
-		(property "Footprint" "A3213ELHLTT"
+		(property "Footprint" "SamacSys_Parts:A3213ELHLTT"
 			(at -60.63 80.01 0)
 			(effects
@@
 			)
 		)
-		(property "Footprint" "SOP65P640X120-16N"
+		(property "Footprint" "SamacSys_Parts:SOP65P640X120-16N"
 			(at 247.65 124.13 0)
 			(effects
@@
 			)
 		)
-		(property "Footprint" "A3213ELHLTT"
+		(property "Footprint" "SamacSys_Parts:A3213ELHLTT"
 			(at 117.17 80.01 0)
 			(effects
@@
 			)
 		)
-		(property "Footprint" "A3213ELHLTT"
+		(property "Footprint" "SamacSys_Parts:A3213ELHLTT"
 			(at 11.76 152.4 0)
 			(effects
