File: ElectroChessboard1/BoardHalls3.kicad_sch (KiCad schematic)
At the start: 18 parts, among them IC37 A3213ELHLT-T, IC38 A3213ELHLT-T, IC39 A3213ELHLT-T, IC40 A3213ELHLT-T, IC41 A3213ELHLT-T, IC42 A3213ELHLT-T, IC43 A3213ELHLT-T, IC44 A3213ELHLT-T, IC45 A3213ELHLT-T, IC46 A3213ELHLT-T, IC47 A3213ELHLT-T, IC48 A3213ELHLT-T, IC49 A3213ELHLT-T, IC50 A3213ELHLT-T, IC51 A3213ELHLT-T, IC52 A3213ELHLT-T, IC53 ADG708BRUZ-REEL7, IC54 ADG708BRUZ-REEL7

Commit message: Corrected footprints 1
Chosen footprints for JLCPCB
I may add USB insterface chip
Parts:
- IC37, IC38, IC39, IC40, IC41, IC42, IC43, IC44, IC45, IC46, IC47, IC48, IC49, IC50, IC51, IC52: footprint A3213ELHLTT -> SamacSys_Parts:A3213ELHLTT
- IC53, IC54: footprint SOP65P640X120-16N -> SamacSys_Parts:SOP65P640X120-16N
Changed lines of the file:
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@@
 			)
 		)
-		(property "Footprint" "A3213ELHLTT"
+		(property "Footprint" "SamacSys_Parts:A3213ELHLTT"
 			(at 42.24 80.01 0)
 			(effects
@@
 			)
 		)
-		(property "Footprint" "A3213ELHLTT"
+		(property "Footprint" "SamacSys_Parts:A3213ELHLTT"
 			(at -63.17 152.4 0)
 			(effects
@@
 			)
 		)
-		(property "Footprint" "A3213ELHLTT"
+		(property "Footprint" "SamacSys_Parts:A3213ELHLTT"
 			(at 118.44 80.01 0)
 			(effects
@@
 			)
 		)
-		(property "Footprint" "SOP65P640X120-16N"
+		(property "Footprint" "SamacSys_Parts:SOP65P640X120-16N"
 			(at 245.11 196.52 0)
 			(effects
@@
 			)
 		)
-		(property "Footprint" "A3213ELHLTT"
+		(property "Footprint" "SamacSys_Parts:A3213ELHLTT"
 			(at 89.23 152.4 0)
 			(effects
@@
 			)
 		)
-		(property "Footprint" "A3213ELHLTT"
+		(property "Footprint" "SamacSys_Parts:A3213ELHLTT"
 			(at 114.63 152.4 0)
 			(effects
@@
 			)
 		)
-		(property "Footprint" "A3213ELHLTT"
+		(property "Footprint" "SamacSys_Parts:A3213ELHLTT"
 			(at -59.36 80.01 0)
 			(effects
@@
 			)
 		)
-		(property "Footprint" "A3213ELHLTT"
+		(property "Footprint" "SamacSys_Parts:A3213ELHLTT"
 			(at -33.96 80.01 0)
 			(effects
@@
 			)
 		)
-		(property "Footprint" "A3213ELHLTT"
+		(property "Footprint" "SamacSys_Parts:A3213ELHLTT"
 			(at 16.84 80.01 0)
 			(effects
@@
 			)
 		)
-		(property "Footprint" "SOP65P640X120-16N"
+		(property "Footprint" "SamacSys_Parts:SOP65P640X120-16N"
 			(at 248.92 124.13 0)
 			(effects
@@
 			)
 		)
-		(property "Footprint" "A3213ELHLTT"
+		(property "Footprint" "SamacSys_Parts:A3213ELHLTT"
 			(at 13.03 152.4 0)
 			(effects
@@
 			)
 		)
-		(property "Footprint" "A3213ELHLTT"
+		(property "Footprint" "SamacSys_Parts:A3213ELHLTT"
 			(at 38.43 152.4 0)
 			(effects
@@
 			)
 		)
-		(property "Footprint" "A3213ELHLTT"
+		(property "Footprint" "SamacSys_Parts:A3213ELHLTT"
 			(at -8.56 80.01 0)
 			(effects
@@
 			)
 		)
-		(property "Footprint" "A3213ELHLTT"
+		(property "Footprint" "SamacSys_Parts:A3213ELHLTT"
 			(at 63.83 152.4 0)
 			(effects
@@
 			)
 		)
-		(property "Footprint" "A3213ELHLTT"
+		(property "Footprint" "SamacSys_Parts:A3213ELHLTT"
 			(at 93.04 80.01 0)
 			(effects
@@
 			)
 		)
-		(property "Footprint" "A3213ELHLTT"
+		(property "Footprint" "SamacSys_Parts:A3213ELHLTT"
 			(at 67.64 80.01 0)
 			(effects
@@
 			)
 		)
-		(property "Footprint" "A3213ELHLTT"
+		(property "Footprint" "SamacSys_Parts:A3213ELHLTT"
 			(at -12.37 152.4 0)
 			(effects
@@
 			)
 		)
-		(property "Footprint" "A3213ELHLTT"
+		(property "Footprint" "SamacSys_Parts:A3213ELHLTT"
 			(at -37.77 152.4 0)
 			(effects
