File: ElectroChessboard1/BoardHalls4.kicad_sch (KiCad schematic)
At the start: 18 parts, among them IC55 A3213ELHLT-T, IC56 A3213ELHLT-T, IC57 A3213ELHLT-T, IC58 A3213ELHLT-T, IC59 A3213ELHLT-T, IC60 A3213ELHLT-T, IC61 A3213ELHLT-T, IC62 A3213ELHLT-T, IC63 A3213ELHLT-T, IC64 A3213ELHLT-T, IC65 A3213ELHLT-T, IC66 A3213ELHLT-T, IC67 A3213ELHLT-T, IC68 A3213ELHLT-T, IC69 A3213ELHLT-T, IC70 A3213ELHLT-T, IC71 ADG708BRUZ-REEL7, IC72 ADG708BRUZ-REEL7

Commit message: Corrected footprints 1
Chosen footprints for JLCPCB
I may add USB insterface chip
Parts:
- IC55, IC56, IC57, IC58, IC59, IC60, IC61, IC62, IC63, IC64, IC65, IC66, IC67, IC68, IC69, IC70: footprint A3213ELHLTT -> SamacSys_Parts:A3213ELHLTT
- IC71, IC72: footprint SOP65P640X120-16N -> SamacSys_Parts:SOP65P640X120-16N
Changed lines of the file:
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@@
 			)
 		)
-		(property "Footprint" "A3213ELHLTT"
+		(property "Footprint" "SamacSys_Parts:A3213ELHLTT"
 			(at -42.85 152.4 0)
 			(effects
@@
 			)
 		)
-		(property "Footprint" "A3213ELHLTT"
+		(property "Footprint" "SamacSys_Parts:A3213ELHLTT"
 			(at 62.56 80.01 0)
 			(effects
@@
 			)
 		)
-		(property "Footprint" "A3213ELHLTT"
+		(property "Footprint" "SamacSys_Parts:A3213ELHLTT"
 			(at 58.75 152.4 0)
 			(effects
@@
 			)
 		)
-		(property "Footprint" "A3213ELHLTT"
+		(property "Footprint" "SamacSys_Parts:A3213ELHLTT"
 			(at 84.15 152.4 0)
 			(effects
@@
 			)
 		)
-		(property "Footprint" "A3213ELHLTT"
+		(property "Footprint" "SamacSys_Parts:A3213ELHLTT"
 			(at 113.36 80.01 0)
 			(effects
@@
 			)
 		)
-		(property "Footprint" "SOP65P640X120-16N"
+		(property "Footprint" "SamacSys_Parts:SOP65P640X120-16N"
 			(at 240.03 196.52 0)
 			(effects
@@
 			)
 		)
-		(property "Footprint" "A3213ELHLTT"
+		(property "Footprint" "SamacSys_Parts:A3213ELHLTT"
 			(at -13.64 80.01 0)
 			(effects
@@
 			)
 		)
-		(property "Footprint" "A3213ELHLTT"
+		(property "Footprint" "SamacSys_Parts:A3213ELHLTT"
 			(at 33.35 152.4 0)
 			(effects
@@
 			)
 		)
-		(property "Footprint" "A3213ELHLTT"
+		(property "Footprint" "SamacSys_Parts:A3213ELHLTT"
 			(at -39.04 80.01 0)
 			(effects
@@
 			)
 		)
-		(property "Footprint" "A3213ELHLTT"
+		(property "Footprint" "SamacSys_Parts:A3213ELHLTT"
 			(at -17.45 152.4 0)
 			(effects
@@
 			)
 		)
-		(property "Footprint" "A3213ELHLTT"
+		(property "Footprint" "SamacSys_Parts:A3213ELHLTT"
 			(at 87.96 80.01 0)
 			(effects
@@
 			)
 		)
-		(property "Footprint" "A3213ELHLTT"
+		(property "Footprint" "SamacSys_Parts:A3213ELHLTT"
 			(at 37.16 80.01 0)
 			(effects
@@
 			)
 		)
-		(property "Footprint" "A3213ELHLTT"
+		(property "Footprint" "SamacSys_Parts:A3213ELHLTT"
 			(at -68.25 152.4 0)
 			(effects
@@
 			)
 		)
-		(property "Footprint" "A3213ELHLTT"
+		(property "Footprint" "SamacSys_Parts:A3213ELHLTT"
 			(at 11.76 80.01 0)
 			(effects
@@
 			)
 		)
-		(property "Footprint" "A3213ELHLTT"
+		(property "Footprint" "SamacSys_Parts:A3213ELHLTT"
 			(at 109.55 152.4 0)
 			(effects
@@
 			)
 		)
-		(property "Footprint" "A3213ELHLTT"
+		(property "Footprint" "SamacSys_Parts:A3213ELHLTT"
 			(at -64.44 80.01 0)
 			(effects
@@
 			)
 		)
-		(property "Footprint" "SOP65P640X120-16N"
+		(property "Footprint" "SamacSys_Parts:SOP65P640X120-16N"
 			(at 243.84 124.13 0)
 			(effects
@@
 			)
 		)
-		(property "Footprint" "A3213ELHLTT"
+		(property "Footprint" "SamacSys_Parts:A3213ELHLTT"
 			(at 7.95 152.4 0)
 			(effects
