File: ElectroChessboard1/board.kicad_sch (KiCad schematic)
At the start: 18 parts, among them IC1 A3213ELHLT-T, IC10 A3213ELHLT-T, IC11 A3213ELHLT-T, IC12 A3213ELHLT-T, IC13 A3213ELHLT-T, IC14 A3213ELHLT-T, IC15 A3213ELHLT-T, IC16 A3213ELHLT-T, IC17 A3213ELHLT-T, IC18 ADG708BRUZ-REEL7, IC2 A3213ELHLT-T, IC3 A3213ELHLT-T, IC4 A3213ELHLT-T, IC5 A3213ELHLT-T, IC6 A3213ELHLT-T, IC7 A3213ELHLT-T, IC8 A3213ELHLT-T, IC9 ADG708BRUZ-REEL7

Commit message: Corrected footprints 1
Chosen footprints for JLCPCB
I may add USB insterface chip
Parts:
- IC1, IC10, IC11, IC12, IC13, IC14, IC15, IC16, IC17, IC2, IC3, IC4, IC5, IC6, IC7, IC8: footprint A3213ELHLTT -> SamacSys_Parts:A3213ELHLTT
- IC18, IC9: footprint SOP65P640X120-16N -> SamacSys_Parts:SOP65P640X120-16N
Changed lines of the file:
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@@
 			)
 		)
-		(property "Footprint" "A3213ELHLTT"
+		(property "Footprint" "SamacSys_Parts:A3213ELHLTT"
 			(at 119.71 147.32 0)
 			(effects
@@
 			)
 		)
-		(property "Footprint" "A3213ELHLTT"
+		(property "Footprint" "SamacSys_Parts:A3213ELHLTT"
 			(at -54.28 74.93 0)
 			(effects
@@
 			)
 		)
-		(property "Footprint" "A3213ELHLTT"
+		(property "Footprint" "SamacSys_Parts:A3213ELHLTT"
 			(at 43.51 147.32 0)
 			(effects
@@
 			)
 		)
-		(property "Footprint" "A3213ELHLTT"
+		(property "Footprint" "SamacSys_Parts:A3213ELHLTT"
 			(at -32.69 147.32 0)
 			(effects
@@
 			)
 		)
-		(property "Footprint" "SOP65P640X120-16N"
+		(property "Footprint" "SamacSys_Parts:SOP65P640X120-16N"
 			(at 254 119.05 0)
 			(effects
@@
 			)
 		)
-		(property "Footprint" "A3213ELHLTT"
+		(property "Footprint" "SamacSys_Parts:A3213ELHLTT"
 			(at 94.31 147.32 0)
 			(effects
@@
 			)
 		)
-		(property "Footprint" "A3213ELHLTT"
+		(property "Footprint" "SamacSys_Parts:A3213ELHLTT"
 			(at 18.11 147.32 0)
 			(effects
@@
 			)
 		)
-		(property "Footprint" "A3213ELHLTT"
+		(property "Footprint" "SamacSys_Parts:A3213ELHLTT"
 			(at 68.91 147.32 0)
 			(effects
@@
 			)
 		)
-		(property "Footprint" "SOP65P640X120-16N"
+		(property "Footprint" "SamacSys_Parts:SOP65P640X120-16N"
 			(at 250.19 191.44 0)
 			(effects
@@
 			)
 		)
-		(property "Footprint" "A3213ELHLTT"
+		(property "Footprint" "SamacSys_Parts:A3213ELHLTT"
 			(at -58.09 147.32 0)
 			(effects
@@
 			)
 		)
-		(property "Footprint" "A3213ELHLTT"
+		(property "Footprint" "SamacSys_Parts:A3213ELHLTT"
 			(at 47.32 74.93 0)
 			(effects
@@
 			)
 		)
-		(property "Footprint" "A3213ELHLTT"
+		(property "Footprint" "SamacSys_Parts:A3213ELHLTT"
 			(at -3.48 74.93 0)
 			(effects
@@
 			)
 		)
-		(property "Footprint" "A3213ELHLTT"
+		(property "Footprint" "SamacSys_Parts:A3213ELHLTT"
 			(at 21.92 74.93 0)
 			(effects
@@
 			)
 		)
-		(property "Footprint" "A3213ELHLTT"
+		(property "Footprint" "SamacSys_Parts:A3213ELHLTT"
 			(at 98.12 74.93 0)
 			(effects
@@
 			)
 		)
-		(property "Footprint" "A3213ELHLTT"
+		(property "Footprint" "SamacSys_Parts:A3213ELHLTT"
 			(at -7.29 147.32 0)
 			(effects
@@
 			)
 		)
-		(property "Footprint" "A3213ELHLTT"
+		(property "Footprint" "SamacSys_Parts:A3213ELHLTT"
 			(at -28.88 74.93 0)
 			(effects
@@
 			)
 		)
-		(property "Footprint" "A3213ELHLTT"
+		(property "Footprint" "SamacSys_Parts:A3213ELHLTT"
 			(at 123.52 74.93 0)
 			(effects
@@
 			)
 		)
-		(property "Footprint" "A3213ELHLTT"
+		(property "Footprint" "SamacSys_Parts:A3213ELHLTT"
 			(at 72.72 74.93 0)
 			(effects
