File: ElectroChessboard1/ElectroChessboard1.kicad_pcb (KiCad board)
At the start: 2 copper layers, 159 parts, among them IC1 A3213ELHLT-T, IC10 A3213ELHLT-T, IC11 A3213ELHLT-T, IC12 A3213ELHLT-T, IC13 A3213ELHLT-T, IC14 A3213ELHLT-T, IC15 A3213ELHLT-T, IC16 A3213ELHLT-T, IC17 A3213ELHLT-T, IC18 ADG708BRUZ-REEL7, IC19 A3213ELHLT-T, IC2 A3213ELHLT-T, IC20 A3213ELHLT-T, IC21 A3213ELHLT-T, IC22 A3213ELHLT-T, IC23 A3213ELHLT-T, IC24 A3213ELHLT-T, IC25 A3213ELHLT-T, IC26 A3213ELHLT-T, IC27 A3213ELHLT-T, IC28 A3213ELHLT-T, IC29 A3213ELHLT-T, IC3 A3213ELHLT-T, IC30 A3213ELHLT-T, IC31 A3213ELHLT-T, IC32 A3213ELHLT-T, IC33 A3213ELHLT-T, IC34 A3213ELHLT-T, IC35 ADG708BRUZ-REEL7, IC36 ADG708BRUZ-REEL7, IC37 A3213ELHLT-T, IC38 A3213ELHLT-T, IC39 A3213ELHLT-T, IC4 A3213ELHLT-T, IC40 A3213ELHLT-T, IC41 A3213ELHLT-T, IC42 A3213ELHLT-T, IC43 A3213ELHLT-T, IC44 A3213ELHLT-T, IC45 A3213ELHLT-T, IC46 A3213ELHLT-T, IC47 A3213ELHLT-T, IC48 A3213ELHLT-T, IC49 A3213ELHLT-T, IC5 A3213ELHLT-T, IC50 A3213ELHLT-T, IC51 A3213ELHLT-T, IC52 A3213ELHLT-T, IC53 ADG708BRUZ-REEL7, IC54 ADG708BRUZ-REEL7, IC55 A3213ELHLT-T, IC56 A3213ELHLT-T, IC57 A3213ELHLT-T, IC58 A3213ELHLT-T, IC59 A3213ELHLT-T, IC6 A3213ELHLT-T, IC60 A3213ELHLT-T, IC61 A3213ELHLT-T, IC62 A3213ELHLT-T, IC63 A3213ELHLT-T, IC64 A3213ELHLT-T, IC65 A3213ELHLT-T, IC66 A3213ELHLT-T, IC67 A3213ELHLT-T, IC68 A3213ELHLT-T, IC69 A3213ELHLT-T, IC7 A3213ELHLT-T, IC70 A3213ELHLT-T, IC71 ADG708BRUZ-REEL7, IC72 ADG708BRUZ-REEL7, IC73 CD74HC154M96, IC74 CD74HC154M96, IC75 DS1307Z+T&R, IC8 A3213ELHLT-T, IC9 ADG708BRUZ-REEL7, J1 USB_B, J2 Conn_01x04_Pin, J3 Conn_01x06, U1 ATmega2560-16A, Y2 XO57CRECNA16M

Commit message: Corrected footprints 1
Chosen footprints for JLCPCB
I may add USB insterface chip
Parts:
- removed C1, C3, C5, C6, C7: KAM21BR71H104JT, SamacSys_Parts:CAPC2012X94N
- removed C2: EEE-1CA100NR, SamacSys_Parts:EEE0GA101SR
- removed C4: GCM21B5G1H103FA16L, SamacSys_Parts:GCM21
- removed D1: PTVS5V0Z1USK, Diode_SMD:Nexperia_DSN1608-2_1.6x0.8mm
- removed D10, D11, D12, D13, D14, D15, D16, D17, D18, D19, D20, D21, D22, D23, D24, D25, D26, D27, D28, D29, D30, D31, D32, D33, D34, D35, D36, D5, D6, D7, D8, D9: LED, LED_SMD:LED_0805_2012Metric
- removed D2: SS12, Diode_SMD:D_SMA
- removed D3: 1N4148, Diode_THT:D_DO-35_SOD27_P7.62mm_Horizontal
- removed F1: 0603L050SLYR, SamacSys_Parts:0603L050SLYR
- removed FB1: 742792040, SamacSys_Parts:BEADC2012X110N
- removed IC1, IC10, IC11, IC12, IC13, IC14, IC15, IC16, IC17, IC19, IC2, IC20, IC21, IC22, IC23, IC24, IC25, IC26, IC27, IC28, IC29, IC3, IC30, IC31, IC32, IC33, IC34, IC37, IC38, IC39, IC4, IC40, IC41, IC42, IC43, IC44, IC45, IC46, IC47, IC48, IC49, IC5, IC50, IC51, IC52, IC55, IC56, IC57, IC58, IC59, IC6, IC60, IC61, IC62, IC63, IC64, IC65, IC66, IC67, IC68, IC69, IC7, IC70, IC8: A3213ELHLT-T, SamacSys_Parts:A3213ELHLTT
- removed IC18, IC35, IC36, IC53, IC54, IC71, IC72, IC9: ADG708BRUZ-REEL7, SamacSys_Parts:SOP65P640X120-16N
- removed IC73, IC74: CD74HC154M96, SamacSys_Parts:SOIC127P1030X265-24N
- removed IC75: DS1307Z+T&R, SamacSys_Parts:SOIC127P600X175-8N
- removed J1: USB_B, Connector_USB:USB_B_Lumberg_2411_02_Horizontal
- removed J2: Conn_01x04_Pin, Connector_PinHeader_1.00mm:PinHeader_1x04_P1.00mm_Vertical
- removed J3: Conn_01x06, Connector_Harwin:Harwin_M20-89006xx_1x06_P2.54mm_Horizontal
- removed R1: ERA-6ARW512V, SamacSys_Parts:ERA6AEB101V
- removed R10, R11, R12, R13, R14, R15, R16, R17, R18, R19, R20, R21, R22, R23, R24, R25, R26, R27, R28, R29, R30, R31, R32, R33, R34, R35, R4, R5, R6, R7, R8, R9: 0402WGF1500TCE, SamacSys_Parts:RESC1005X40N
- removed R2, R3: 0402WGF1002TCE, SamacSys_Parts:RESC1005X40N
- removed U1: ATmega2560-16A, Package_QFP:TQFP-100_14x14mm_P0.5mm
- removed Y2: XO57CRECNA16M, SamacSys_Parts:XO57CRECNA16M

Commit message: Added FT232RL
Ready for PCB design
Parts:
- added C1: CL10C220JB8NNNC, SamacSys_Parts:CAPC1608X90N, F.Cu at (136.1, 45.1)
- added C10: CL10B104KC8NNNC, SamacSys_Parts:CAPC1608X90N, F.Cu at (180.5, 110.0)
- added C3: CL10C220JB8NNNC, SamacSys_Parts:CAPC1608X90N, F.Cu at (136.1, 47.4)
- added C4: CL10B104KC8NNNC, SamacSys_Parts:CAPC1608X90N, F.Cu at (136.1, 49.7)
- added C5: CL10B104KC8NNNC, SamacSys_Parts:CAPC1608X90N, F.Cu at (180.5, 105.4)
- added C6: CL10B104KC8NNNC, SamacSys_Parts:CAPC1608X90N, F.Cu at (183.7, 70.2)
- added C7: CL10B104KC8NNNC, SamacSys_Parts:CAPC1608X90N, F.Cu at (158.6, 70.2)
- added C8: CL10B104KC8NNNC, SamacSys_Parts:CAPC1608X90N, F.Cu at (180.5, 107.7)
- added C9: C_Polarized, Capacitor_SMD:CP_Elec_4x5.4, F.Cu at (163.8, 113.2)
- added D1: ESD5Z5V0, SamacSys_Parts:SODFL1608X70N, F.Cu at (183.9, 112.0)
- added D10: LED, LED_SMD:LED_0805_2012Metric, F.Cu at (175.7, 48.5)
- added D11: LED, LED_SMD:LED_0805_2012Metric, F.Cu at (175.7, 51.6)
- added D12: LED, LED_SMD:LED_0805_2012Metric, F.Cu at (175.7, 54.6)
- added D13: LED, LED_SMD:LED_0805_2012Metric, F.Cu at (180.2, 45.5)
- added D14: LED, LED_SMD:LED_0805_2012Metric, F.Cu at (180.2, 48.5)
- added D15: LED, LED_SMD:LED_0805_2012Metric, F.Cu at (180.2, 51.6)
- added D16: LED, LED_SMD:LED_0805_2012Metric, F.Cu at (180.2, 54.6)
- added D17: LED, LED_SMD:LED_0805_2012Metric, F.Cu at (184.6, 45.5)
- added D18: LED, LED_SMD:LED_0805_2012Metric, F.Cu at (184.6, 48.5)
- added D19: LED, LED_SMD:LED_0805_2012Metric, F.Cu at (184.6, 51.6)
- added D2: SS12, Diode_SMD:D_SMA, F.Cu at (171.7, 112.5)
- added D20: LED, LED_SMD:LED_0805_2012Metric, F.Cu at (184.6, 54.6)
- added D21: LED, LED_SMD:LED_0805_2012Metric, F.Cu at (146.1, 45.5)
- added D22: LED, LED_SMD:LED_0805_2012Metric, F.Cu at (146.1, 48.5)
- added D23: LED, LED_SMD:LED_0805_2012Metric, F.Cu at (146.1, 51.6)
- added D24: LED, LED_SMD:LED_0805_2012Metric, F.Cu at (146.1, 54.6)
- added D25: LED, LED_SMD:LED_0805_2012Metric, F.Cu at (150.6, 45.5)
- added D26: LED, LED_SMD:LED_0805_2012Metric, F.Cu at (150.6, 48.5)
- added D27: LED, LED_SMD:LED_0805_2012Metric, F.Cu at (150.6, 51.6)
- added D28: LED, LED_SMD:LED_0805_2012Metric, F.Cu at (150.6, 54.6)
- added D29: LED, LED_SMD:LED_0805_2012Metric, F.Cu at (155.0, 45.5)
- added D3: 1N4148, Diode_SMD:D_SOD-123, F.Cu at (137.3, 52.5)
- added D30: LED, LED_SMD:LED_0805_2012Metric, F.Cu at (155.0, 48.5)
- added D31: LED, LED_SMD:LED_0805_2012Metric, F.Cu at (155.0, 51.6)
- added D32: LED, LED_SMD:LED_0805_2012Metric, F.Cu at (155.0, 54.6)
- added D33: LED, LED_SMD:LED_0805_2012Metric, F.Cu at (159.5, 45.5)
- added D34: LED, LED_SMD:LED_0805_2012Metric, F.Cu at (159.5, 48.5)
- added D35: LED, LED_SMD:LED_0805_2012Metric, F.Cu at (159.5, 51.6)
- added D36: LED, LED_SMD:LED_0805_2012Metric, F.Cu at (159.5, 54.6)
- added D5: LED, LED_SMD:LED_0805_2012Metric, F.Cu at (171.3, 45.5)
- added D6: LED, LED_SMD:LED_0805_2012Metric, F.Cu at (171.3, 48.5)
- added D7: LED, LED_SMD:LED_0805_2012Metric, F.Cu at (171.3, 51.6)
- added D8: LED, LED_SMD:LED_0805_2012Metric, F.Cu at (171.3, 54.6)
- added D9: LED, LED_SMD:LED_0805_2012Metric, F.Cu at (175.7, 45.5)
- added F1: 0603L050SLYR, SamacSys_Parts:0603L050SLYR, F.Cu at (185.2, 106.3)
- added FB1: GZ1608D601TF, SamacSys_Parts:BEADC1608X95N, F.Cu at (184.2, 109.7)
- added IC1: A3213ELHLT-T, SamacSys_Parts:A3213ELHLTT, F.Cu at (92.5, 123.5)
- added IC10: A3213ELHLT-T, SamacSys_Parts:A3213ELHLTT, F.Cu at (92.5, 136.5)
- added IC11: A3213ELHLT-T, SamacSys_Parts:A3213ELHLTT, F.Cu at (98.6, 136.5)
- added IC12: A3213ELHLT-T, SamacSys_Parts:A3213ELHLTT, F.Cu at (104.7, 136.5)
- added IC13: A3213ELHLT-T, SamacSys_Parts:A3213ELHLTT, F.Cu at (110.8, 136.5)
- added IC14: A3213ELHLT-T, SamacSys_Parts:A3213ELHLTT, F.Cu at (92.5, 143.0)
- added IC15: A3213ELHLT-T, SamacSys_Parts:A3213ELHLTT, F.Cu at (98.6, 143.0)
- added IC16: A3213ELHLT-T, SamacSys_Parts:A3213ELHLTT, F.Cu at (104.7, 143.0)
- added IC17: A3213ELHLT-T, SamacSys_Parts:A3213ELHLTT, F.Cu at (110.8, 143.0)
- added IC18: ADG708BRUZ-REEL7, SamacSys_Parts:SOP65P640X120-16N, F.Cu at (118.2, 130.4)
- added IC19: A3213ELHLT-T, SamacSys_Parts:A3213ELHLTT, F.Cu at (92.5, 95.5)
- added IC2: A3213ELHLT-T, SamacSys_Parts:A3213ELHLTT, F.Cu at (98.6, 123.5)
- added IC20: A3213ELHLT-T, SamacSys_Parts:A3213ELHLTT, F.Cu at (98.6, 95.5)
- added IC21: A3213ELHLT-T, SamacSys_Parts:A3213ELHLTT, F.Cu at (104.7, 95.5)
- added IC22: A3213ELHLT-T, SamacSys_Parts:A3213ELHLTT, F.Cu at (110.8, 95.5)
- added IC23: A3213ELHLT-T, SamacSys_Parts:A3213ELHLTT, F.Cu at (92.5, 102.0)
- added IC24: A3213ELHLT-T, SamacSys_Parts:A3213ELHLTT, F.Cu at (98.6, 102.0)
- added IC25: A3213ELHLT-T, SamacSys_Parts:A3213ELHLTT, F.Cu at (104.7, 102.0)
- added IC26: A3213ELHLT-T, SamacSys_Parts:A3213ELHLTT, F.Cu at (110.8, 102.0)
- added IC27: A3213ELHLT-T, SamacSys_Parts:A3213ELHLTT, F.Cu at (92.5, 108.5)
- added IC28: A3213ELHLT-T, SamacSys_Parts:A3213ELHLTT, F.Cu at (98.6, 108.5)
- added IC29: A3213ELHLT-T, SamacSys_Parts:A3213ELHLTT, F.Cu at (104.7, 108.5)
- added IC3: A3213ELHLT-T, SamacSys_Parts:A3213ELHLTT, F.Cu at (104.7, 123.5)
- added IC30: A3213ELHLT-T, SamacSys_Parts:A3213ELHLTT, F.Cu at (110.8, 108.5)
- added IC31: A3213ELHLT-T, SamacSys_Parts:A3213ELHLTT, F.Cu at (92.5, 115.0)
- added IC32: A3213ELHLT-T, SamacSys_Parts:A3213ELHLTT, F.Cu at (98.6, 115.0)
- added IC33: A3213ELHLT-T, SamacSys_Parts:A3213ELHLTT, F.Cu at (104.7, 115.0)
- added IC34: A3213ELHLT-T, SamacSys_Parts:A3213ELHLTT, F.Cu at (110.8, 115.0)
- added IC35: ADG708BRUZ-REEL7, SamacSys_Parts:SOP65P640X120-16N, F.Cu at (118.2, 95.7)
- added IC36: ADG708BRUZ-REEL7, SamacSys_Parts:SOP65P640X120-16N, F.Cu at (118.2, 102.5)
- added IC37: A3213ELHLT-T, SamacSys_Parts:A3213ELHLTT, F.Cu at (127.7, 95.5)
- added IC38: A3213ELHLT-T, SamacSys_Parts:A3213ELHLTT, F.Cu at (133.8, 95.5)
- added IC39: A3213ELHLT-T, SamacSys_Parts:A3213ELHLTT, F.Cu at (139.9, 95.5)
- added IC4: A3213ELHLT-T, SamacSys_Parts:A3213ELHLTT, F.Cu at (110.8, 123.5)
- added IC40: A3213ELHLT-T, SamacSys_Parts:A3213ELHLTT, F.Cu at (146.0, 95.5)
- added IC41: A3213ELHLT-T, SamacSys_Parts:A3213ELHLTT, F.Cu at (127.7, 102.0)
- added IC42: A3213ELHLT-T, SamacSys_Parts:A3213ELHLTT, F.Cu at (133.8, 102.0)
- added IC43: A3213ELHLT-T, SamacSys_Parts:A3213ELHLTT, F.Cu at (139.9, 102.0)
- added IC44: A3213ELHLT-T, SamacSys_Parts:A3213ELHLTT, F.Cu at (146.0, 102.0)
- added IC45: A3213ELHLT-T, SamacSys_Parts:A3213ELHLTT, F.Cu at (127.7, 108.5)
- added IC46: A3213ELHLT-T, SamacSys_Parts:A3213ELHLTT, F.Cu at (133.8, 108.5)
- added IC47: A3213ELHLT-T, SamacSys_Parts:A3213ELHLTT, F.Cu at (139.9, 108.5)
- added IC48: A3213ELHLT-T, SamacSys_Parts:A3213ELHLTT, F.Cu at (146.0, 108.5)
- added IC49: A3213ELHLT-T, SamacSys_Parts:A3213ELHLTT, F.Cu at (127.7, 115.0)
- added IC5: A3213ELHLT-T, SamacSys_Parts:A3213ELHLTT, F.Cu at (92.5, 130.0)
- added IC50: A3213ELHLT-T, SamacSys_Parts:A3213ELHLTT, F.Cu at (133.8, 115.0)
- added IC51: A3213ELHLT-T, SamacSys_Parts:A3213ELHLTT, F.Cu at (139.9, 115.0)
- added IC52: A3213ELHLT-T, SamacSys_Parts:A3213ELHLTT, F.Cu at (146.0, 115.0)
- added IC53: ADG708BRUZ-REEL7, SamacSys_Parts:SOP65P640X120-16N, F.Cu at (153.5, 95.7)
- added IC54: ADG708BRUZ-REEL7, SamacSys_Parts:SOP65P640X120-16N, F.Cu at (153.5, 102.5)
- added IC55: A3213ELHLT-T, SamacSys_Parts:A3213ELHLTT, F.Cu at (127.7, 123.5)
- added IC56: A3213ELHLT-T, SamacSys_Parts:A3213ELHLTT, F.Cu at (133.8, 123.5)
- added IC57: A3213ELHLT-T, SamacSys_Parts:A3213ELHLTT, F.Cu at (139.9, 123.5)
- added IC58: A3213ELHLT-T, SamacSys_Parts:A3213ELHLTT, F.Cu at (146.0, 123.5)
- added IC59: A3213ELHLT-T, SamacSys_Parts:A3213ELHLTT, F.Cu at (127.7, 130.0)
- added IC6: A3213ELHLT-T, SamacSys_Parts:A3213ELHLTT, F.Cu at (98.6, 130.0)
- added IC60: A3213ELHLT-T, SamacSys_Parts:A3213ELHLTT, F.Cu at (133.8, 130.0)
- added IC61: A3213ELHLT-T, SamacSys_Parts:A3213ELHLTT, F.Cu at (139.9, 130.0)
- added IC62: A3213ELHLT-T, SamacSys_Parts:A3213ELHLTT, F.Cu at (146.0, 130.0)
- added IC63: A3213ELHLT-T, SamacSys_Parts:A3213ELHLTT, F.Cu at (127.7, 136.5)
- added IC64: A3213ELHLT-T, SamacSys_Parts:A3213ELHLTT, F.Cu at (133.8, 136.5)
- added IC65: A3213ELHLT-T, SamacSys_Parts:A3213ELHLTT, F.Cu at (139.9, 136.5)
- added IC66: A3213ELHLT-T, SamacSys_Parts:A3213ELHLTT, F.Cu at (146.0, 136.5)
- added IC67: A3213ELHLT-T, SamacSys_Parts:A3213ELHLTT, F.Cu at (127.7, 143.0)
- added IC68: A3213ELHLT-T, SamacSys_Parts:A3213ELHLTT, F.Cu at (133.8, 143.0)
- added IC69: A3213ELHLT-T, SamacSys_Parts:A3213ELHLTT, F.Cu at (139.9, 143.0)
- added IC7: A3213ELHLT-T, SamacSys_Parts:A3213ELHLTT, F.Cu at (104.7, 130.0)
- added IC70: A3213ELHLT-T, SamacSys_Parts:A3213ELHLTT, F.Cu at (146.0, 143.0)
- added IC71: ADG708BRUZ-REEL7, SamacSys_Parts:SOP65P640X120-16N, F.Cu at (153.5, 123.7)
- added IC72: ADG708BRUZ-REEL7, SamacSys_Parts:SOP65P640X120-16N, F.Cu at (153.5, 130.4)
- added IC73: CD74HC154M96, SamacSys_Parts:SOIC127P1030X265-24N, F.Cu at (175.5, 64.7)
- added IC74: CD74HC154M96, SamacSys_Parts:SOIC127P1030X265-24N, F.Cu at (150.4, 64.7)
- added IC75: DS1307Z+T&R, SamacSys_Parts:SOIC127P600X175-8N, F.Cu at (130.1, 47.2)
- added IC8: A3213ELHLT-T, SamacSys_Parts:A3213ELHLTT, F.Cu at (110.8, 130.0)
- added IC9: ADG708BRUZ-REEL7, SamacSys_Parts:SOP65P640X120-16N, F.Cu at (118.2, 123.7)
- added J1: USB_B, Connector_USB:USB_B_Lumberg_2411_02_Horizontal, F.Cu at (162.5, 100.0)
- added J3: Conn_01x04_Pin, Connector_PinSocket_1.00mm:PinSocket_1x04_P1.00mm_Vertical_SMD_Pin1Left, F.Cu at (128.8, 53.8)
- added J5: Conn_01x06, Connector_PinSocket_1.00mm:PinSocket_1x06_P1.00mm_Vertical_SMD_Pin1Right, F.Cu at (126.5, 86.0)
- added J6: Conn_01x06, Connector_PinSocket_1.00mm:PinSocket_1x06_P1.00mm_Vertical_SMD_Pin1Right, F.Cu at (132.5, 86.0)
- added R1: R, Resistor_SMD:R_0402_1005Metric, F.Cu at (139.3, 49.3)
- added R10: 0402WGF1500TCE, SamacSys_Parts:RESC1005X40N, F.Cu at (187.1, 59.4)
- added R11: 0402WGF1500TCE, SamacSys_Parts:RESC1005X40N, F.Cu at (187.1, 61.5)
- added R12: 0402WGF1500TCE, SamacSys_Parts:RESC1005X40N, F.Cu at (187.1, 63.7)
- added R13: 0402WGF1500TCE, SamacSys_Parts:RESC1005X40N, F.Cu at (187.1, 65.8)
- added R14: 0402WGF1500TCE, SamacSys_Parts:RESC1005X40N, F.Cu at (187.1, 68.0)
- added R15: 0402WGF1500TCE, SamacSys_Parts:RESC1005X40N, F.Cu at (190.5, 57.2)
- added R16: 0402WGF1500TCE, SamacSys_Parts:RESC1005X40N, F.Cu at (190.5, 59.4)
- added R17: 0402WGF1500TCE, SamacSys_Parts:RESC1005X40N, F.Cu at (190.5, 61.5)
- added R18: 0402WGF1500TCE, SamacSys_Parts:RESC1005X40N, F.Cu at (190.5, 63.7)
- added R19: 0402WGF1500TCE, SamacSys_Parts:RESC1005X40N, F.Cu at (190.5, 65.8)
- added R2: 0402WGF1002TCE, SamacSys_Parts:RESC1005X40N, F.Cu at (183.7, 57.2)
- added R20: 0402WGF1500TCE, SamacSys_Parts:RESC1005X40N, F.Cu at (158.5, 59.4)
- added R21: 0402WGF1500TCE, SamacSys_Parts:RESC1005X40N, F.Cu at (158.5, 61.5)
- added R22: 0402WGF1500TCE, SamacSys_Parts:RESC1005X40N, F.Cu at (158.5, 63.7)
- added R23: 0402WGF1500TCE, SamacSys_Parts:RESC1005X40N, F.Cu at (158.5, 65.8)
- added R24: 0402WGF1500TCE, SamacSys_Parts:RESC1005X40N, F.Cu at (158.5, 68.0)
- added R25: 0402WGF1500TCE, SamacSys_Parts:RESC1005X40N, F.Cu at (161.9, 57.2)
- added R26: 0402WGF1500TCE, SamacSys_Parts:RESC1005X40N, F.Cu at (161.9, 59.4)
- added R27: 0402WGF1500TCE, SamacSys_Parts:RESC1005X40N, F.Cu at (161.9, 61.5)
- added R28: 0402WGF1500TCE, SamacSys_Parts:RESC1005X40N, F.Cu at (161.9, 63.7)
- added R29: 0402WGF1500TCE, SamacSys_Parts:RESC1005X40N, F.Cu at (161.9, 65.8)
- added R3: 0402WGF1002TCE, SamacSys_Parts:RESC1005X40N, F.Cu at (158.5, 57.2)
- added R30: 0402WGF1500TCE, SamacSys_Parts:RESC1005X40N, F.Cu at (161.9, 68.0)
- added R31: 0402WGF1500TCE, SamacSys_Parts:RESC1005X40N, F.Cu at (165.3, 57.2)
- added R32: 0402WGF1500TCE, SamacSys_Parts:RESC1005X40N, F.Cu at (165.3, 59.4)
- added R33: 0402WGF1500TCE, SamacSys_Parts:RESC1005X40N, F.Cu at (165.3, 61.5)
- added R34: 0402WGF1500TCE, SamacSys_Parts:RESC1005X40N, F.Cu at (165.3, 63.7)
- added R35: 0402WGF1500TCE, SamacSys_Parts:RESC1005X40N, F.Cu at (165.3, 65.8)
- added R38: RC0402FR-074K7L, SamacSys_Parts:RESC1005X40N, F.Cu at (139.6, 45.0)
- added R39: RC0402FR-074K7L, SamacSys_Parts:RESC1005X40N, F.Cu at (139.6, 47.2)
- added R4: 0402WGF1500TCE, SamacSys_Parts:RESC1005X40N, F.Cu at (183.7, 59.4)
- added R5: 0402WGF1500TCE, SamacSys_Parts:RESC1005X40N, F.Cu at (183.7, 61.5)
- added R6: 0402WGF1500TCE, SamacSys_Parts:RESC1005X40N, F.Cu at (183.7, 63.7)
- added R7: 0402WGF1500TCE, SamacSys_Parts:RESC1005X40N, F.Cu at (183.7, 65.8)
- added R8: 0402WGF1500TCE, SamacSys_Parts:RESC1005X40N, F.Cu at (183.7, 68.0)
- added R9: 0402WGF1500TCE, SamacSys_Parts:RESC1005X40N, F.Cu at (187.1, 57.2)
- added S1: EVQ-9P105M, SamacSys_Parts:EVQ9P105M, F.Cu at (94.0, 50.5)
- added S2: EVQ-9P105M, SamacSys_Parts:EVQ9P105M, F.Cu at (103.1, 50.5)
- added S3: EVQ-9P105M, SamacSys_Parts:EVQ9P105M, F.Cu at (112.2, 50.5)
- added S4: EVQ-9P105M, SamacSys_Parts:EVQ9P105M, F.Cu at (121.3, 50.5)
- added U1: ATmega2560-16A, Package_QFP:TQFP-100_14x14mm_P0.5mm, F.Cu at (132.7, 66.2)
- added U2: 1027, SamacSys_Parts:1027, F.Cu at (114.7, 72.5)
- added U3: FT232RL, Package_SO:SSOP-28_5.3x10.2mm_P0.65mm, F.Cu at (184.0, 98.2)
- added Y1: Crystal, Crystal:Crystal_SMD_HC49-SD, F.Cu at (130.9, 78.5)
- added Y3: Crystal, Crystal:Crystal_C38-LF_D3.0mm_L8.0mm_Vertical, F.Cu at (137.0, 84.2)
