File: ElectroChessboard1/ElectroChessboard1.kicad_pcb (KiCad board)
At the start: 2 copper layers, 171 parts, among them IC1 A3213ELHLT-T, IC10 A3213ELHLT-T, IC11 A3213ELHLT-T, IC12 A3213ELHLT-T, IC13 A3213ELHLT-T, IC14 A3213ELHLT-T, IC15 A3213ELHLT-T, IC16 A3213ELHLT-T, IC17 A3213ELHLT-T, IC18 ADG708BRUZ-REEL7, IC19 A3213ELHLT-T, IC2 A3213ELHLT-T, IC20 A3213ELHLT-T, IC21 A3213ELHLT-T, IC22 A3213ELHLT-T, IC23 A3213ELHLT-T, IC24 A3213ELHLT-T, IC25 A3213ELHLT-T, IC26 A3213ELHLT-T, IC27 A3213ELHLT-T, IC28 A3213ELHLT-T, IC29 A3213ELHLT-T, IC3 A3213ELHLT-T, IC30 A3213ELHLT-T, IC31 A3213ELHLT-T, IC32 A3213ELHLT-T, IC33 A3213ELHLT-T, IC34 A3213ELHLT-T, IC35 ADG708BRUZ-REEL7, IC36 ADG708BRUZ-REEL7, IC37 A3213ELHLT-T, IC38 A3213ELHLT-T, IC39 A3213ELHLT-T, IC4 A3213ELHLT-T, IC40 A3213ELHLT-T, IC41 A3213ELHLT-T, IC42 A3213ELHLT-T, IC43 A3213ELHLT-T, IC44 A3213ELHLT-T, IC45 A3213ELHLT-T, IC46 A3213ELHLT-T, IC47 A3213ELHLT-T, IC48 A3213ELHLT-T, IC49 A3213ELHLT-T, IC5 A3213ELHLT-T, IC50 A3213ELHLT-T, IC51 A3213ELHLT-T, IC52 A3213ELHLT-T, IC53 ADG708BRUZ-REEL7, IC54 ADG708BRUZ-REEL7, IC55 A3213ELHLT-T, IC56 A3213ELHLT-T, IC57 A3213ELHLT-T, IC58 A3213ELHLT-T, IC59 A3213ELHLT-T, IC6 A3213ELHLT-T, IC60 A3213ELHLT-T, IC61 A3213ELHLT-T, IC62 A3213ELHLT-T, IC63 A3213ELHLT-T, IC64 A3213ELHLT-T, IC65 A3213ELHLT-T, IC66 A3213ELHLT-T, IC67 A3213ELHLT-T, IC68 A3213ELHLT-T, IC69 A3213ELHLT-T, IC7 A3213ELHLT-T, IC70 A3213ELHLT-T, IC71 ADG708BRUZ-REEL7, IC72 ADG708BRUZ-REEL7, IC73 CD74HC154M96, IC74 CD74HC154M96, IC75 DS1307Z+T&R, IC8 A3213ELHLT-T, IC9 ADG708BRUZ-REEL7, J1 USB_B, J3 Conn_01x04_Pin, J5 Conn_01x06, J6 Conn_01x06, U1 ATmega2560-16A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

Commit message: Chessboard layout
drawn with silkscreen
Other:
- board outline added: 326 x 392.5 mm

Commit message: Hall detectors on chessboard
I put them
Parts:
- moved IC71 404.6 mm to (448.1, 401.0)
- moved IC69 385.1 mm to (426.8, 399.9)
- moved IC53 382.9 mm to (449.2, 338.8)
- moved IC35 380.1 mm to (450.8, 279.7)
- moved IC72 379.8 mm to (448.6, 369.5)
- moved IC67 372.0 mm to (396.8, 399.9)
- moved IC51 364.6 mm to (426.8, 339.9)
- moved IC36 363.1 mm to (450.8, 248.2)
- moved IC33 361.9 mm to (426.8, 279.9)
- moved IC54 361.9 mm to (449.6, 310.5)
- moved IC70 361.0 mm to (426.8, 369.9)
- moved IC49 350.7 mm to (396.8, 339.9)
- moved IC65 347.7 mm to (366.8, 399.9)
- moved IC68 347.4 mm to (396.8, 369.9)
- moved IC31 346.1 mm to (396.8, 279.9)
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
Commit message: Hall sensors in middle of fields
.
Parts:
- moved C10 225.8 mm to (-43.3, 140.0)
- moved C5 225.8 mm to (-43.3, 135.5)
- moved C6 225.8 mm to (-40.0, 100.2)
- moved C8 225.8 mm to (-43.3, 137.8)
- moved D2 225.8 mm to (-52.0, 142.6)
- moved D25 225.8 mm to (-73.2, 75.5)
- moved D26 225.8 mm to (-73.2, 78.6)
- moved D27 225.8 mm to (-73.2, 81.6)
- moved D28 225.8 mm to (-73.2, 84.7)
- moved IC74 225.8 mm to (-73.4, 94.8)
- moved R1 225.8 mm to (-84.4, 79.3)
- moved R15 225.8 mm to (-33.3, 87.2)
- moved R16 225.8 mm to (-33.3, 89.4)
- moved R17 225.8 mm to (-33.3, 91.5)
- moved R18 225.8 mm to (-33.3, 93.7)
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Other:
- board size 326 x 392.5 mm -> 308.2 x 311.2 mm

Commit message: update
Parts:
- moved D28 268.4 mm to (134.2, 254.9), turned to -90 degrees
- moved D27 252.1 mm to (134.2, 224.8), turned to -90 degrees
- moved D36 239.5 mm to (104.2, 254.8), turned to -90 degrees
- moved D26 238.0 mm to (134.5, 194.8), turned to -90 degrees
- moved D25 226.0 mm to (134.5, 164.6), turned to -90 degrees
- moved D35 221.2 mm to (104.2, 224.8), turned to -90 degrees
- moved D24 217.9 mm to (134.5, 134.6), turned to -90 degrees
- moved D21 214.6 mm to (134.8, 44.8), turned to -90 degrees
- moved D13 214.5 mm to (74.2, 254.8), turned to -90 degrees
- moved D23 213.4 mm to (134.5, 104.7), turned to -90 degrees
- moved D22 212.2 mm to (134.5, 74.7), turned to -90 degrees
- moved D34 204.9 mm to (104.5, 194.8), turned to -90 degrees
- moved D5 203.7 mm to (44.2, 254.8), turned to -90 degrees
- moved D33 190.9 mm to (104.5, 164.8), turned to -90 degrees
- moved D14 188.0 mm to (74.2, 225.1), turned to -90 degrees
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
Commit message: Chessboard done
Other parts left to place. Also, I changed some wiring in schematic, changing what was connected to RX TX1
Parts:
- added C11: CL10B104KC8NNNC, SamacSys_Parts:CAPC1608X90N, F.Cu at (185.5, 293.2)
- added C12: CL10B104KC8NNNC, SamacSys_Parts:CAPC1608X90N, F.Cu at (245.8, 292.5)
- added D37: LED, LED_SMD:LED_0805_2012Metric, F.Cu at (194.8, 45.1)
- added D38: LED, LED_SMD:LED_0805_2012Metric, F.Cu at (194.8, 74.6)
- added D39: LED, LED_SMD:LED_0805_2012Metric, F.Cu at (194.5, 104.8)
- added D40: LED, LED_SMD:LED_0805_2012Metric, F.Cu at (194.5, 134.8)
- added D41: LED, LED_SMD:LED_0805_2012Metric, F.Cu at (194.5, 164.6)
- added D42: LED, LED_SMD:LED_0805_2012Metric, F.Cu at (194.5, 195.1)
- added D43: LED, LED_SMD:LED_0805_2012Metric, F.Cu at (194.2, 224.8)
- added D44: LED, LED_SMD:LED_0805_2012Metric, F.Cu at (194.2, 254.8)
- added D45: LED, LED_SMD:LED_0805_2012Metric, F.Cu at (164.5, 45.1)
- added D46: LED, LED_SMD:LED_0805_2012Metric, F.Cu at (164.5, 74.6)
- added D47: LED, LED_SMD:LED_0805_2012Metric, F.Cu at (164.5, 104.8)
- added D48: LED, LED_SMD:LED_0805_2012Metric, F.Cu at (164.5, 134.8)
- added D49: LED, LED_SMD:LED_0805_2012Metric, F.Cu at (164.5, 164.8)
- added D50: LED, LED_SMD:LED_0805_2012Metric, F.Cu at (164.5, 194.8)
- added D51: LED, LED_SMD:LED_0805_2012Metric, F.Cu at (164.2, 224.8)
- added D52: LED, LED_SMD:LED_0805_2012Metric, F.Cu at (164.2, 254.8)
- added D53: LED, LED_SMD:LED_0805_2012Metric, F.Cu at (255.0, 44.8)
- added D54: LED, LED_SMD:LED_0805_2012Metric, F.Cu at (254.8, 74.7)
- added D55: LED, LED_SMD:LED_0805_2012Metric, F.Cu at (254.5, 104.8)
- added D56: LED, LED_SMD:LED_0805_2012Metric, F.Cu at (254.5, 134.8)
- added D57: LED, LED_SMD:LED_0805_2012Metric, F.Cu at (254.5, 164.6)
- added D58: LED, LED_SMD:LED_0805_2012Metric, F.Cu at (254.5, 194.6)
- added D59: LED, LED_SMD:LED_0805_2012Metric, F.Cu at (254.2, 224.8)
- added D60: LED, LED_SMD:LED_0805_2012Metric, F.Cu at (254.2, 254.8)
- added D61: LED, LED_SMD:LED_0805_2012Metric, F.Cu at (225.0, 45.3)
- added D62: LED, LED_SMD:LED_0805_2012Metric, F.Cu at (225.0, 74.6)
- added D63: LED, LED_SMD:LED_0805_2012Metric, F.Cu at (224.5, 104.8)
- added D64: LED, LED_SMD:LED_0805_2012Metric, F.Cu at (224.5, 134.6)
- added D65: LED, LED_SMD:LED_0805_2012Metric, F.Cu at (224.5, 164.8)
- added D66: LED, LED_SMD:LED_0805_2012Metric, F.Cu at (224.5, 194.7)
- added D67: LED, LED_SMD:LED_0805_2012Metric, F.Cu at (224.2, 224.8)
- added D68: LED, LED_SMD:LED_0805_2012Metric, F.Cu at (224.2, 254.7)
- added IC76: CD74HC154M96, SamacSys_Parts:SOIC127P1030X265-24N, F.Cu at (183.0, 283.3)
- added IC77: CD74HC154M96, SamacSys_Parts:SOIC127P1030X265-24N, F.Cu at (243.7, 282.3)
- added R36: 0402WGF1002TCE, SamacSys_Parts:RESC1005X40N, F.Cu at (181.6, 293.2)
- added R37: 0402WGF1500TCE, SamacSys_Parts:RESC1005X40N, F.Cu at (194.8, 49.0)
- added R40: 0402WGF1500TCE, SamacSys_Parts:RESC1005X40N, F.Cu at (194.8, 78.5)
- added R41: 0402WGF1500TCE, SamacSys_Parts:RESC1005X40N, F.Cu at (194.5, 108.8)
- added R42: 0402WGF1500TCE, SamacSys_Parts:RESC1005X40N, F.Cu at (194.5, 138.8)
- added R43: 0402WGF1500TCE, SamacSys_Parts:RESC1005X40N, F.Cu at (194.5, 168.7)
- added R44: 0402WGF1500TCE, SamacSys_Parts:RESC1005X40N, F.Cu at (194.5, 199.2)
- added R45: 0402WGF1500TCE, SamacSys_Parts:RESC1005X40N, F.Cu at (194.2, 228.7)
- added R46: 0402WGF1500TCE, SamacSys_Parts:RESC1005X40N, F.Cu at (194.2, 258.7)
- added R47: 0402WGF1500TCE, SamacSys_Parts:RESC1005X40N, F.Cu at (164.5, 49.0)
- added R48: 0402WGF1500TCE, SamacSys_Parts:RESC1005X40N, F.Cu at (164.5, 78.3)
- added R49: 0402WGF1500TCE, SamacSys_Parts:RESC1005X40N, F.Cu at (164.5, 108.8)
- added R50: 0402WGF1500TCE, SamacSys_Parts:RESC1005X40N, F.Cu at (164.5, 138.8)
- added R51: 0402WGF1500TCE, SamacSys_Parts:RESC1005X40N, F.Cu at (164.5, 168.8)
- added R52: 0402WGF1500TCE, SamacSys_Parts:RESC1005X40N, F.Cu at (164.5, 198.8)
- added R53: 0402WGF1500TCE, SamacSys_Parts:RESC1005X40N, F.Cu at (164.2, 228.9)
- added R54: 0402WGF1500TCE, SamacSys_Parts:RESC1005X40N, F.Cu at (164.2, 259.1)
- added R55: 0402WGF1002TCE, SamacSys_Parts:RESC1005X40N, F.Cu at (241.2, 292.5)
- added R56: 0402WGF1500TCE, SamacSys_Parts:RESC1005X40N, F.Cu at (255.0, 48.8)
- added R57: 0402WGF1500TCE, SamacSys_Parts:RESC1005X40N, F.Cu at (254.8, 78.8)
- added R58: 0402WGF1500TCE, SamacSys_Parts:RESC1005X40N, F.Cu at (254.5, 108.8)
- added R59: 0402WGF1500TCE, SamacSys_Parts:RESC1005X40N, F.Cu at (254.5, 138.7)
- added R60: 0402WGF1500TCE, SamacSys_Parts:RESC1005X40N, F.Cu at (254.5, 168.7)
- added R61: 0402WGF1500TCE, SamacSys_Parts:RESC1005X40N, F.Cu at (254.5, 198.6)
- added R62: 0402WGF1500TCE, SamacSys_Parts:RESC1005X40N, F.Cu at (254.2, 228.8)
- added R63: 0402WGF1500TCE, SamacSys_Parts:RESC1005X40N, F.Cu at (254.2, 258.8)
- added R64: 0402WGF1500TCE, SamacSys_Parts:RESC1005X40N, F.Cu at (225.0, 49.3)
- added R65: 0402WGF1500TCE, SamacSys_Parts:RESC1005X40N, F.Cu at (225.0, 78.5)
- added R66: 0402WGF1500TCE, SamacSys_Parts:RESC1005X40N, F.Cu at (224.5, 109.0)
- added R67: 0402WGF1500TCE, SamacSys_Parts:RESC1005X40N, F.Cu at (224.5, 138.6)
- added R68: 0402WGF1500TCE, SamacSys_Parts:RESC1005X40N, F.Cu at (224.5, 168.8)
- added R69: 0402WGF1500TCE, SamacSys_Parts:RESC1005X40N, F.Cu at (224.5, 198.6)
- added R70: 0402WGF1500TCE, SamacSys_Parts:RESC1005X40N, F.Cu at (224.2, 228.8)
- added R71: 0402WGF1500TCE, SamacSys_Parts:RESC1005X40N, F.Cu at (224.2, 258.4)
- moved R3 279.4 mm to (125.0, 292.0)
- moved IC74 271.3 mm to (122.5, 282.5)
- moved C7 267.1 mm to (120.8, 292.0)
- moved R27 257.8 mm to (134.2, 258.9), turned to -90 degrees
- moved R26 240.5 mm to (134.2, 228.7), turned to -90 degrees
- moved R35 230.1 mm to (104.2, 258.6), turned to -90 degrees
- moved R2 227.1 mm to (56.7, 292.8)
- moved R25 225.9 mm to (134.5, 198.9), turned to -90 degrees
- moved C6 218.0 mm to (61.8, 293.0)
- moved IC73 216.7 mm to (60.3, 282.3)
- moved R24 211.9 mm to (134.5, 168.8), turned to -90 degrees
- moved R34 211.5 mm to (104.2, 228.8), turned to -90 degrees
- moved R23 204.3 mm to (134.5, 138.7), turned to -90 degrees
- moved R20 204.0 mm to (134.8, 49.0), turned to -90 degrees
- moved R22 200.3 mm to (134.5, 108.8), turned to -90 degrees
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Connections:
- U1 pad 12: unconnected-(U1-PH0-Pad12) -> LED_A1_3
- U1 pad 13: unconnected-(U1-PH1-Pad13) -> LED_A0_3
- U1 pad 63: unconnected-(U1-PJ0-Pad63) -> LED_A3_3
- U1 pad 64: unconnected-(U1-PJ1-Pad64) -> LED_A3_2
- U1 pad 82: unconnected-(U1-PK7-Pad82) -> LED_A1_2
- U1 pad 83: unconnected-(U1-PK6-Pad83) -> LED_A0_2
- U1 pad 84: unconnected-(U1-PK5-Pad84) -> LED_EN_3
- U1 pad 85: unconnected-(U1-PK4-Pad85) -> LED_EN_2
Routing:
- net Net-(D52-A): track 0.00 -> 2.75 mm
- net Net-(D25-A): track 0.00 -> 2.75 mm
- net Net-(D63-A): track 0.00 -> 2.65 mm
- net Net-(D57-A): track 0.00 -> 2.65 mm
- net Net-(D51-A): track 0.00 -> 2.65 mm
- net Net-(D42-A): track 0.00 -> 2.65 mm
- net Net-(D41-A): track 0.00 -> 2.65 mm
- net Net-(D31-A): track 0.00 -> 2.65 mm
- net Net-(D26-A): track 0.00 -> 2.65 mm
- net Net-(D24-A): track 0.00 -> 2.65 mm
- net Net-(D54-A): track 0.00 -> 2.62 mm
- net Net-(D23-A): track 0.00 -> 2.62 mm
- net Net-(D22-A): track 0.00 -> 2.62 mm
- net Net-(D28-A): track 0.00 -> 2.52 mm
- net Net-(D8-A): track 0.00 -> 2.50 mm
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
Commit message: Added oled
.
Parts:
- moved J3 396.8 mm to (296.3, 150.2), turned to 180 degrees
Other:
- board size 308.2 x 311.2 mm -> 305.2 x 309 mm
- board text added: "OLED 27x27mm"
Changed lines of the file:
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@@
 	)
 	(paper "User" 390 390)
+	(title_block
+		(title "ElectroChessboard")
+		(company "Wojciech B")
+		(comment 1 "Electronic chessboard")
+		(comment 2 "Elektroniczna szachownica")
+	)
 	(layers
 		(0 "F.Cu" signal)
@@
 	(footprint "Connector_PinSocket_1.00mm:PinSocket_1x04_P1.00mm_Vertical_SMD_Pin1Left"
 		(layer "F.Cu")
-		(at -94.91 83.84)
+		(at 296.275 150.25 180)
 		(descr "surface-mounted straight socket strip, 1x04, 1.00mm pitch, single row, style 1 (pin 1 left) (https://gct.co/files/drawings/bc070.pdf), script generated")
 		(tags "Surface mounted socket strip SMD 1x04 1.00mm single row style1 pin1 left")
@@
 		)
 		(property "Datasheet" ""
-			(at 0 0 0)
+			(at 0 0 180)
 			(unlocked yes)
 			(layer "F.Fab")
@@
 		)
 		(property "Description" "Generic connector, single row, 01x04, script generated"
-			(at 0 0 0)
+			(at 0 0 180)
 			(unlocked yes)
 			(layer "F.Fab")
@@
 		(attr smd)
 		(fp_line
-			(start -1.89 -2.01)
-			(end -0.81 -2.01)
+			(start 0.81 2.01)
+			(end 0.81 2.31)
 			(stroke
 				(width 0.12)
@@
 		)
 		(fp_line
-			(start -0.81 -2.31)
-			(end -0.81 -2.01)
+			(start 0.81 0.01)
+			(end 0.81 0.99)
 			(stroke
 				(width 0.12)
@@
 		)
 		(fp_line
-			(start -0.81 -2.31)
-			(end 0.81 -2.31)
+			(start 0.81 -2.31)
+			(end 0.81 -1.01)
 			(stroke
 				(width 0.12)
@@
 		)
 		(fp_line
-			(start -0.81 -0.99)
-			(end -0.81 -0.01)
+			(start -0.81 2.31)
+			(end 0.81 2.31)
 			(stroke
 				(width 0.12)
@@
 		)
 		(fp_line
-			(start -0.81 2.31)
-			(end 0.81 2.31)
+			(start -0.81 -0.99)
+			(end -0.81 -0.01)
 			(stroke
 				(width 0.12)
@@
 		)
 		(fp_line
-			(start 0.81 -2.31)
-			(end 0.81 -1.01)
+			(start -0.81 -2.31)
+			(end 0.81 -2.31)
 			(stroke
 				(width 0.12)
@@
 		)
 		(fp_line
-			(start 0.81 0.01)
-			(end 0.81 0.99)
+			(start -0.81 -2.31)
+			(end -0.81 -2.01)
 			(stroke
 				(width 0.12)
@@
 		)
 		(fp_line
-			(start 0.81 2.01)
-			(end 0.81 2.31)
+			(start -1.89 -2.01)
+			(end -0.81 -2.01)
 			(stroke
 				(width 0.12)
@@
 		)
 		(fp_line
-			(start -2.45 -2.75)
-			(end 2.45 -2.75)
+			(start 2.45 2.75)
+			(end -2.45 2.75)
 			(stroke
 				(width 0.05)
@@
 		)
 		(fp_line
-			(start -2.45 2.75)
-			(end -2.45 -2.75)
+			(start 2.45 -2.75)
+			(end 2.45 2.75)
 			(stroke
 				(width 0.05)
@@
 		)
 		(fp_line
-			(start 2.45 -2.75)
-			(end 2.45 2.75)
+			(start -2.45 2.75)
+			(end -2.45 -2.75)
 			(stroke
 				(width 0.05)
@@
 		)
 		(fp_line
-			(start 2.45 2.75)
-			(end -2.45 2.75)
+			(start -2.45 -2.75)
+			(end 2.45 -2.75)
 			(stroke
 				(width 0.05)
@@
 		)
 		(fp_line
-			(start -1.45 -1.65)
-			(end -0.75 -1.65)
+			(start 1.45 1.65)
+			(end 0.75 1.65)
 			(stroke
 				(width 0.1)
@@
 		)
 		(fp_line
-			(start -1.45 -1.35)
-			(end -1.45 -1.65)
+			(start 1.45 1.35)
+			(end 1.45 1.65)
 			(stroke
 				(width 0.1)
@@
 		)
 		(fp_line
-			(start -1.45 0.35)
-			(end -0.75 0.35)
+			(start 1.45 -0.35)
+			(end 0.75 -0.35)
 			(stroke
 				(width 0.1)
@@
 		)
 		(fp_line
-			(start -1.45 0.65)
-			(end -1.45 0.35)
+			(start 1.45 -0.65)
+			(end 1.45 -0.35)
 			(stroke
 				(width 0.1)
@@
 		)
 		(fp_line
-			(start -0.75 -1.875)
-			(end -0.375 -2.25)
+			(start 0.75 2.25)
+			(end -0.75 2.25)
 			(stroke
 				(width 0.1)
@@
 		)
 		(fp_line
-			(start -0.75 -1.35)
-			(end -1.45 -1.35)
+			(start 0.75 1.35)
+			(end 1.45 1.35)
 			(stroke
 				(width 0.1)
@@
 		)
 		(fp_line
-			(start -0.75 0.65)
-			(end -1.45 0.65)
+			(start 0.75 -0.65)
+			(end 1.45 -0.65)
 			(stroke
 				(width 0.1)
@@
 		)
 		(fp_line
-			(start -0.75 2.25)
-			(end -0.75 -1.875)
+			(start 0.75 -2.25)
+			(end 0.75 2.25)
 			(stroke
 				(width 0.1)
@@
 		)
 		(fp_line
-			(start 0.75 -2.25)
-			(end 0.75 2.25)
+			(start -0.75 2.25)
+			(end -0.75 -1.875)
 			(stroke
 				(width 0.1)
@@
 		)
 		(fp_line
-			(start 0.75 -0.65)
-			(end 1.45 -0.65)
+			(start -0.75 0.65)
+			(end -1.45 0.65)
 			(stroke
 				(width 0.1)
@@
 		)
 		(fp_line
-			(start 0.75 1.35)
-			(end 1.45 1.35)
+			(start -0.75 -1.35)
+			(end -1.45 -1.35)
 			(stroke
 				(width 0.1)
@@
 		)
 		(fp_line
-			(start 0.75 2.25)
-			(end -0.75 2.25)
+			(start -0.75 -1.875)
+			(end -0.375 -2.25)
 			(stroke
 				(width 0.1)
@@
 		)
 		(fp_line
-			(start 1.45 -0.65)
-			(end 1.45 -0.35)
+			(start -1.45 0.65)
+			(end -1.45 0.35)
 			(stroke
 				(width 0.1)
@@
 		)
 		(fp_line
-			(start 1.45 -0.35)
-			(end 0.75 -0.35)
+			(start -1.45 0.35)
+			(end -0.75 0.35)
 			(stroke
 				(width 0.1)
@@
 		)
 		(fp_line
-			(start 1.45 1.35)
-			(end 1.45 1.65)
+			(start -1.45 -1.35)
+			(end -1.45 -1.65)
 			(stroke
 				(width 0.1)
@@
 		)
 		(fp_line
-			(start 1.45 1.65)
-			(end 0.75 1.65)
+			(start -1.45 -1.65)
+			(end -0.75 -1.65)
 			(stroke
 				(width 0.1)
@@
 		)
 		(pad "1" smd rect
-			(at -0.975 -1.5)
+			(at -0.975 -1.5 180)
 			(size 1.95 0.5)
 			(layers "F.Cu" "F.Mask" "F.Paste")
@@
 		)
 		(pad "2" smd rect
-			(at 0.975 -0.5)
+			(at 0.975 -0.5 180)
 			(size 1.95 0.5)
 			(layers "F.Cu" "F.Mask" "F.Paste")
@@
 		)
 		(pad "3" smd rect
-			(at -0.975 0.5)
+			(at -0.975 0.5 180)
 			(size 1.95 0.5)
 			(layers "F.Cu" "F.Mask" "F.Paste")
@@
 		)
 		(pad "4" smd rect
-			(at 0.975 1.5)
+			(at 0.975 1.5 180)
 			(size 1.95 0.5)
 			(layers "F.Cu" "F.Mask" "F.Paste")
@@
 	)
 	(gr_rect
+		(start 293.75 136.75)
+		(end 324.5 163.75)
+		(stroke
+			(width 0.1)
+			(type default)
+		)
+		(fill no)
+		(layer "F.SilkS")
+	)
+	(gr_rect
 		(start 124.5 180.25)
 		(end 154.5 210.25)
@@
 	)
 	(gr_rect
-		(start 21.25 17.75)
+		(start 24.25 20)
 		(end 329.5 329)
 		(stroke
@@
 		(layer "Edge.Cuts")
 	)
+	(gr_text "OLED 27x27mm"
+		(at 305.75 155.75 90)
+		(layer "F.SilkS")
+		(effects
+			(font
+				(size 1 1)
+				(thickness 0.1)
+			)
+			(justify left bottom)
+		)
+	)
 	(segment

Commit message: Fixed pins
Now footprints of pins match
Parts:
- J3: footprint Connector_PinSocket_1.00mm:PinSocket_1x04_P1.00mm_Vertical_SMD_Pin1Left -> Connector_PinSocket_1.27mm:PinSocket_1x04_P1.27mm_Vertical_SMD_Pin1Right
- J5, J6: footprint Connector_PinSocket_1.00mm:PinSocket_1x06_P1.00mm_Vertical_SMD_Pin1Right -> Connector_PinSocket_2.00mm:PinSocket_1x06_P2.00mm_Vertical_SMD_Pin1Right
- moved J3 0.23 mm to (296.5, 150.2)

Commit message: Big part layout done
Microcontroller, mux/demux layout and of course wiring left. Also changed footprint of the SD card module pins.
Parts:
- J5: footprint Connector_PinSocket_2.00mm:PinSocket_1x06_P2.00mm_Vertical_SMD_Pin1Right -> Connector_PinSocket_2.54mm:PinSocket_1x06_P2.54mm_Horizontal
- moved S1 436.1 mm to (304.1, 124.8), turned to -90 degrees
- moved S3 426.6 mm to (304.1, 176.3), turned to -90 degrees
- moved S2 425.7 mm to (304.1, 108.8), turned to -90 degrees
- moved S4 421.7 mm to (304.1, 192.3), turned to -90 degrees
- moved J5 281.1 mm to (110.0, 305.8)
- moved C6 50.2 mm to (111.8, 296.8)
- moved R2 50.2 mm to (106.7, 296.5)
- moved IC73 49.4 mm to (109.5, 285.6)
- moved C7 11.0 mm to (129.8, 298.2)
- moved R3 11.0 mm to (133.9, 298.2)
- moved IC74 10.7 mm to (132.0, 287.3)
- moved U2 9.27 mm to (-117.5, 98.8)
- moved IC35 5.68 mm to (278.1, 134.8), turned to 90 degrees
- moved IC36 5.48 mm to (278.1, 105.3), turned to 90 degrees
- moved IC18 5.31 mm to (278.1, 75.3), turned to 90 degrees
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Other:
- board size 305.2 x 309 mm -> 306.2 x 314.8 mm
- board text added: "SD card reader"
